File: SandKrux.kicad_pcb (KiCad board)
At the start: 2 copper layers, 58.3 x 98.2 mm, 174 parts, among them CN2 1.25mm-2P socket, IC1 TROPIC01_chip, Q1 S8050, Q2 SI2301CDS-T1-GE3, SW1 TL3330AF130QG, SW2 TL3330AF130QG, SW3 TL3330AF130QG, SW4 TL3330AF130QG, SW5 TL3330AF130QG, U1 K210_C913414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

Commit message: muito trabalho to quase acabando
Parts:
- removed Q2: SI2301CDS-T1-GE3, PCM_JLCPCB:Q_SOT-89
- removed R32, R33: 1.5K, Resistor_SMD:R_0201_0603Metric
- added C10: 10uF, Capacitor_SMD:C_0201_0603Metric, F.Cu at (96.3, 114.6)
- added C11: 10uF, Capacitor_SMD:C_0201_0603Metric, F.Cu at (96.3, 115.4)
- added C12: 10uF, Capacitor_SMD:C_0201_0603Metric, F.Cu at (100.5, 108.3)
- added C13: 10uF, Capacitor_SMD:C_0201_0603Metric, F.Cu at (100.5, 109.1)
- added C14: 10uF, Capacitor_SMD:C_0201_0603Metric, F.Cu at (100.5, 109.9)
- added C15: 10uF, Capacitor_SMD:C_0201_0603Metric, F.Cu at (100.5, 110.7)
- added C16: 10uF, Capacitor_SMD:C_0201_0603Metric, F.Cu at (117.5, 109.0)
- added C17: 10uF, Capacitor_SMD:C_0201_0603Metric, F.Cu at (117.5, 108.2)
- added C18: 100nF, Capacitor_SMD:C_0201_0603Metric, F.Cu at (117.5, 107.4)
- added C19: 100nF, Capacitor_SMD:C_0201_0603Metric, F.Cu at (117.5, 106.6)
- added C4: 100nF, Capacitor_SMD:C_0201_0603Metric, F.Cu at (109.7, 117.1)
- added C5: 100nF, Capacitor_SMD:C_0201_0603Metric, F.Cu at (109.7, 117.9)
- added C6: 100nF, Capacitor_SMD:C_0201_0603Metric, F.Cu at (109.7, 118.8)
- added C7: 100nF, Capacitor_SMD:C_0201_0603Metric, F.Cu at (109.7, 119.6)
- added C8: 10uF, Capacitor_SMD:C_0201_0603Metric, F.Cu at (96.3, 113.0)
- added C9: 10uF, Capacitor_SMD:C_0201_0603Metric, F.Cu at (96.3, 113.8)
- added U3: XC6206-3.3V, easyeda2kicad:SSOT-3_L2.9-W1.6-P0.95-LS2.8-BR, F.Cu at (111.8, 139.2)
- moved TP1 7.92 mm to (124.3, 113.5)
- moved JP1 0.80 mm to (114.2, 118.2)
- moved JP2 0.80 mm to (111.7, 118.2)
Connections:
- U12 pad 76: unconnected-(U12-Pad76) -> GND
- U12 pad 77: unconnected-(U12-Pad77) -> GND
Routing:
- net GND: track 465.8 -> 488.2 mm, vias 148 -> 152
- net +3.3V: track 100.1 -> 109.4 mm
- net /3V3: track 215.0 -> 219.6 mm
- net /k210/0V9: track 93.4 -> 95.5 mm
- net /VCC_1V83V3: track 21.9 -> 23.5 mm
- net /k210/DVP_VSYNC: track 14.8 -> 15.6 mm
- net /k210/1V8: track 47.6 -> 48.3 mm
- net /k210/Vb: track 8.51 -> 9.10 mm
- net /k210/DVP_HSYNC: track 14.5 -> 15.1 mm
- net /k210/26M_OUT: track 1.29 -> 0.93 mm, vias 1 -> 0
- net /k210/IO_22: track 0.32 -> 0.02 mm, vias 1 -> 0
