File: SandKrux.kicad_pcb (KiCad board)
At the start: 2 copper layers, 58.3 x 98.2 mm, 188 parts, among them CN2 1.25mm-2P socket, IC1 TROPIC01_chip, Q1 S8050, SW1 TL3330AF130QG, SW2 TL3330AF130QG, SW3 TL3330AF130QG, SW4 TL3330AF130QG, SW5 TL3330AF130QG, U1 K210_C913414, U10 AXP173_C3345106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

Commit message: CH552T
Parts:
- removed C69, C70: 10uF, Capacitor_SMD:C_0201_0603Metric
- removed C71, C72: 18pF, Capacitor_SMD:C_0201_0603Metric
- removed LED1, LED2: KT-0603R, easyeda2kicad:LED0603-RD
- removed R45: 1.5, Resistor_SMD:R_0201_0603Metric
- removed R46, R49: 1.5K, Resistor_SMD:R_0201_0603Metric
- removed R47, R48, R50, R51, R52: 22R, Resistor_SMD:R_0201_0603Metric
- removed R53, R56: 5.1K, Resistor_SMD:R_0201_0603Metric
- removed R54: 10K, Resistor_SMD:R_0201_0603Metric
- removed R55: NC, Resistor_SMD:R_0201_0603Metric
- removed U11: GD32F150G8U6, easyeda2kicad:WQFN-28_L4.0-W4.0-P0.40-BL-EP
- removed X2: X322526MMB4SI, PCM_JLCPCB:CRYSTAL-SMD_4P-L3.2-W2.5-BL
- added C77: 22uF, PCM_JLCPCB:C_0603, F.Cu at (131.8, 175.0)
- added C79: 10uF, PCM_JLCPCB:C_0603, F.Cu at (130.6, 175.0)
- added R32: 1kΩ, PCM_JLCPCB:R_0603, F.Cu at (126.4, 163.6)
- added R33: 1kΩ, PCM_JLCPCB:R_0603, F.Cu at (127.8, 162.0)
- added U13: CH552T, easyeda2kicad:TSSOP-20_L6.5-W4.4-P0.65-LS6.4-BL, F.Cu at (128.5, 169.5)
- moved REF** 81.7 mm to (92.9, 99.6)
- moved TP3 1.00 mm to (89.2, 177.2)
- moved TP2 0.64 mm to (89.4, 172.2)
- moved C54 0.64 mm to (99.7, 170.3)
- moved C68 0.64 mm to (101.4, 170.3)
- moved C53 0.64 mm to (98.8, 170.3)
- moved C66 0.64 mm to (102.3, 170.3)
- moved C67 0.64 mm to (100.5, 170.3)
- moved U7 0.45 mm to (121.4, 111.7)
Connections:
- net /RST renamed /CH552_P1.0
- U1 pad H11: /k210/IO_4 -> /ISP_RX
- U1 pad H12: /k210/IO_5 -> /CH552_RX0
- U12 pad 40: unconnected-(U12-Pad40) -> /CH552_RX0
- U12 pad 42: unconnected-(U12-Pad42) -> /ISP_RX
- USB1 pad A6: /USB_D+ -> /USBDP
- USB1 pad A7: /USB_D- -> /USBDM
- USB1 pad B6: /USB_D+ -> /USBDP
- USB1 pad B7: /USB_D- -> /USBDM
Routing:
- net /USB_D-: track 103.4 -> 20.2 mm, vias 3 -> 2
- net /USB_D+: track 100.6 -> 20.0 mm, vias 3 -> 2
- net /CH552_RX0: track 0.00 -> 72.8 mm, vias 0 -> 4
- net /ISP_RX: track 0.00 -> 71.8 mm, vias 0 -> 4
- net GND: track 488.2 -> 546.2 mm, vias 152 -> 95
- net /BOOT: track 18.4 -> 70.4 mm, vias 2 -> 4
- net /3V3: track 219.6 -> 169.0 mm, vias 5 -> 4
- net /CH552_P1.0: track 80.2 -> 123.2 mm, vias 3 -> 5
- net /USBDM: track 0.00 -> 22.2 mm
- net /USBDP: track 0.00 -> 19.2 mm
- net /5V_USB: track 70.0 -> 88.4 mm
- net /5V: track 150.2 -> 138.5 mm, vias 11 -> 7
- net +3.3V: track 109.4 -> 100.0 mm
- net /24M_IN: track 7.06 -> 0.00 mm
- net Net-(FPC3-Pad20): track 21.3 -> 15.6 mm
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