File: SandKrux.kicad_sch (KiCad schematic)
At the start: 121 parts, among them CN2 1.25mm-2P socket, IC1 TROPIC01_chip, Q1 S8050, Q2 SI2301CDS-T1-GE3, SW1 TL3330AF130QG, SW2 TL3330AF130QG, SW3 TL3330AF130QG, SW4 TL3330AF130QG, SW5 TL3330AF130QG, U10 AXP173_C3345106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

Commit message: muito trabalho to quase acabando
Parts:
- removed Q2: SI2301CDS-T1-GE3, PCM_JLCPCB:Q_SOT-89, symbol PCM_JLCPCB-Transistors:PMOS,SI2301CDS-T1-GE3
- removed R32, R33: 1.5K, Resistor_SMD:R_0201_0603Metric, symbol Device:R
- added U3: XC6206-3.3V, easyeda2kicad:SSOT-3_L2.9-W1.6-P0.95-LS2.8-BR, symbol easyeda2kicad:XC6206-3.3V
Connections:
- net 3V3: now also U3.3 (VIN)
- net LCD_BACKLIGHT: now also U3.2 (VOUT)
- net at R14.2: now also U3.1 (VSS)
- no-connect marks 35 -> 33
Other:
- sheet k210 ports: added none; removed DVP_D6, DVP_D7, DVP_HSYNC, DVP_PCLK, DVP_PWDN, DVP_RST, DVP_SCL, DVP_SDA, DVP_VSYNC, DVP_XCLK
- moved on the sheet: H1, H2, H3, H4
