File: SandKrux.kicad_sch (KiCad schematic)
At the start: 104 parts, among them CN2 1.25mm-2P socket, IC1 TROPIC01_chip, Q1 S8050, SW1 TL3330AF130QG, SW2 TL3330AF130QG, SW3 TL3330AF130QG, SW4 TL3330AF130QG, SW5 TL3330AF130QG, U10 AXP173_C3345106, U13 CH552T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

Commit message: ajuste de esquematico e posicionamento de componentes
Parts:
- added JP3, JP4: SolderJumper_2_Bridged, Jumper:SolderJumper-2_P1.3mm_Bridged_RoundedPad1.0x1.5mm, symbol Jumper:SolderJumper_2_Bridged
Connections:
- net USBDM: now also JP4.1 (A); no longer U13.15 (P3.7/UDM)
- net USBDP: now also JP3.1 (A); no longer U13.14 (P3.6/UDP)
- new net: JP3.2 (B), U13.14 (P3.6/UDP)
- new net: JP4.2 (B), U13.15 (P3.7/UDM)
Other:
- note added: "BOTAO"
- note added: "k210"
- moved on the sheet: C73, C74, C75, C77, C79, H1, H2, H3, H4, IC1, R32, R33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

Commit message: CNC AND PRINTER
Parts:
- removed CN2: 1.25mm-2P socket, easyeda2kicad:CONN-SMD_1.25T-2P, symbol easyeda2kicad:1.25mm-2Psocket
- added CN2: SM02B-PASS-TBT(LF)(SN), easyeda2kicad:CONN-SMD_SM02B-PASS-TBT, symbol easyeda2kicad:SM02B-PASS-TBT(LF)(SN)
- added CN3: 1.25mm-2P socket, easyeda2kicad:CONN-SMD_1.25T-2P, symbol easyeda2kicad:1.25mm-2Psocket
Connections:
- net GND: now also CN2.2, CN2.3, CN2.4, CN3.0, CN3.2
- net VBAT: now also CN3.1
- new net PRINTER: CN2.1
Other:
- sheet k210 ports: added PRINTER; removed none
- note added: "CNC AND PRINTER"
