File: untitled.kicad_sch (KiCad schematic)
At the start: 66 parts, among them U1 K210_C913414, U12 PCIE-67P42H, U4 XC6206P182MR_C347373, U5 GD25LQ128EWIGR, U6 TMI7003C, U7 SGM803-TXN3/TR_C5152602, U8 XC6206P302MR_C347375, X1 X322526MMB4SI

Commit message: CNC AND PRINTER
Connections:
- net IO_7 is gone; now on net PRINTER: U1.G12 (IO_7)
- net PRINTER: now reaches U12.71
- no-connect marks 42 -> 41
Changed lines of the file:
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@@
 	)
 	(no_connect
-		(at 340.36 176.53)
-	)
-	(no_connect
 		(at 340.36 146.05)
 	)
@@
 	(wire
 		(pts
+			(xy 340.36 176.53) (xy 354.33 176.53)
+		)
+		(stroke
+			(width 0)
+			(type default)
+		)
+	)
+	(wire
+		(pts
 			(xy 88.9 49.53) (xy 96.52 49.53)
 		)
@@
 		)
 	)
+	(label "IO_7"
+		(at 347.98 176.53 0)
+		(effects
+			(font
+				(size 1.27 1.27)
+			)
+			(justify left bottom)
+		)
+	)
 	(label "3V3"
 		(at 251.46 29.21 0)
@@
 		)
 	)
+	(hierarchical_label "PRINTER"
+		(shape bidirectional)
+		(at 354.33 176.53 0)
+		(effects
+			(font
+				(size 1.27 1.27)
+			)
+			(justify left)
+		)
+	)
